File: New layout/ESP32-IoT-Board-ChipAnt.kicad_pcb (KiCad board)
At the start: 4 copper layers, 23.9 x 27.2 mm, 50 parts, among them IC1 MIC5528-3.3YMT-T5, IC2 ESP32-C3FH4, IC3 ADXL335BCPZ-RL, J1 LiPo Battery, J2 USB_B_Micro, Q1 FDN340P, U1 USBLC6-2SC6, U2 MCP73831-2-OT, U3 MCP9700AT-ETT, Y1 40 Mhz Crystal

Commit message: Final
Parts:
- moved D1 0.25 mm to (146.2, 98.1)
- moved R1 0.22 mm to (149.0, 97.8)
Routing:
- net VBUS: track 27.6 -> 25.0 mm
- net Net-(C1-Pad1): track 11.3 -> 10.7 mm
